File: kicad/core/sense.kicad_sch (KiCad schematic)
At the start: 9 parts, among them U1 TLV3501AID, U2 74AHC74

Commit message: Docs updated to match physical core layout.
Connections:
- net YA66 renamed YA65
Changed lines of the file:
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@@
 	(title_block
 		(title "Sense")
-		(comment 1 "TLV3501 / 74AHC74 latch (beads on ferrite_beads)")
+		(comment 1 "TLV3501 / 74AHC74; 1k from YA65 to SENSE_P and YB66 to SENSE_N")
 	)
 	(text "SENSE — Sense amp / latch\nClamps: BAT54S rot90 — +3V3 (K) above, GND (A) below\nC1/C2 at U1; C3/C4 at U2; blocks spaced for hand placement"
@@
 		)
 	)
-	(label "YA66"
+	(hierarchical_label "YA65"
+		(shape passive)
 		(at 46.99 63.5 0)
 		(effects
