File: kicad/core/core.kicad_sch (KiCad schematic)
At the start: 0 parts

Commit message: Prove the 2×2 access cycle from the address pins through decode, drive, and the sense latch.
Three current sinks, the diode matrix, and drive groups 0--7 are on the schematic. The four-core decks are the gate; weave inductance is still an open input.
Parts:
- added J400, J401, J402, J403, J404, J405, J406, J407, J408, J409, J410, J411, J412, J413, J414, J415, J416: PIO, Connector_PinHeader_2.54mm:PinHeader_1x01_P2.54mm_Vertical, symbol Connector:Conn_01x01
- added J500, J501, J502, J503, J504, J505, J506, J507, J508, J509, J510, J511, J512, J513, J514, J515, J516, J517, J518, J519, J520, J521, J522, J523, J524, J525, J526, J527, J528, J529, J530, J531, J532, J533, J534, J535, J536, J537, J538, J539, J540, J541, J542, J543, J544, J545, J546, J547, J548, J549, J550, J551, J552, J553, J554, J555, J556, J557, J558, J559, J560, J561, J562, J563, J564, J565, J566, J567, J568, J569, J570, J571, J572, J573, J574, J575, J576, J577, J578, J579, J580, J581, J582, J583, J584, J585, J586, J587, J588, J589, J590, J591, J592, J593, J594, J595, J596, J597, J598, J599, J600, J601, J602, J603, J604, J605, J606, J607, J608, J609, J610, J611, J612, J613, J614, J615, J616, J617, J618, J619, J620, J621, J622, J623, J624, J625, J626, J627, J628, J629, J630, J631, J632, J633, J634, J635, J636, J637, J638, J639, J640, J641, J642, J643, J644, J645, J646, J647, J648, J649, J650, J651, J652, J653, J654, J655, J656, J657, J658, J659, J660, J661, J662, J663, J664, J665, J666, J667, J668, J669, J670, J671, J672, J673, J674, J675, J676, J677, J678, J679, J680, J681, J682, J683, J684, J685, J686, J687, J688, J689, J690, J691, J692, J693, J694, J695, J696, J697, J698, J699, J700, J701, J702, J703, J704, J705, J706, J707, J708, J709, J710, J711, J712, J713, J714, J715, J716, J717, J718, J719, J720, J721, J722, J723, J724, J725, J726, J727, J728, J729, J730, J731, J732, J733, J734, J735, J736, J737, J738, J739, J740, J741, J742, J743, J744, J745, J746, J747, J748, J749, J750, J751, J752, J753, J754, J755: Edge, Connector_PinHeader_2.54mm:PinHeader_1x01_P2.54mm_Vertical, symbol Connector:Conn_01x01
Connections:
- net ADDR_XH0: now also J400.1 (Pin_1)
- net ADDR_XH1: now also J401.1 (Pin_1)
- net ADDR_XH2: now also J402.1 (Pin_1)
- net ADDR_XL0: now also J403.1 (Pin_1)
- net ADDR_XL1: now also J404.1 (Pin_1)
- net ADDR_XL2: now also J405.1 (Pin_1)
- net ADDR_YH0: now also J406.1 (Pin_1)
- net ADDR_YH1: now also J407.1 (Pin_1)
- net ADDR_YH2: now also J408.1 (Pin_1)
- net ADDR_YL0: now also J409.1 (Pin_1)
- net ADDR_YL1: now also J410.1 (Pin_1)
- net ADDR_YL2: now also J411.1 (Pin_1)
- net DEC_EN: now also J412.1 (Pin_1)
- net FWD_EN_n: now also J413.1 (Pin_1)
- net REV_EN_n: now also J414.1 (Pin_1)
- net XA0: now also J500.1 (Pin_1)
- net XA1: now also J501.1 (Pin_1)
- net XB0: now also J564.1 (Pin_1)
- net XB1: now also J565.1 (Pin_1)
- net YA0: now also J628.1 (Pin_1)
- net YA1: now also J629.1 (Pin_1)
- net YB0: now also J692.1 (Pin_1)
- net YB1: now also J693.1 (Pin_1)
- new net INH_EN_n: J415.1 (Pin_1)
- new net SENSE_STROBE: J416.1 (Pin_1)
- new net XA10: J510.1 (Pin_1)
- new net XA11: J511.1 (Pin_1)
- new net XA12: J512.1 (Pin_1)
- new net XA13: J513.1 (Pin_1)
- new net XA14: J514.1 (Pin_1)
- new net XA15: J515.1 (Pin_1)
- new net XA16: J516.1 (Pin_1)
- new net XA17: J517.1 (Pin_1)
- new net XA18: J518.1 (Pin_1)
- new net XA19: J519.1 (Pin_1)
- new net XA2: J502.1 (Pin_1)
- new net XA20: J520.1 (Pin_1)
- new net XA21: J521.1 (Pin_1)
- new net XA22: J522.1 (Pin_1)
- new net XA23: J523.1 (Pin_1)
- new net XA24: J524.1 (Pin_1)
- new net XA25: J525.1 (Pin_1)
- new net XA26: J526.1 (Pin_1)
- new net XA27: J527.1 (Pin_1)
- new net XA28: J528.1 (Pin_1)
- new net XA29: J529.1 (Pin_1)
- new net XA3: J503.1 (Pin_1)
- new net XA30: J530.1 (Pin_1)
- new net XA31: J531.1 (Pin_1)
- new net XA32: J532.1 (Pin_1)
- new net XA33: J533.1 (Pin_1)
- new net XA34: J534.1 (Pin_1)
- new net XA35: J535.1 (Pin_1)
- new net XA36: J536.1 (Pin_1)
- new net XA37: J537.1 (Pin_1)
- new net XA38: J538.1 (Pin_1)
- new net XA39: J539.1 (Pin_1)
- new net XA4: J504.1 (Pin_1)
- new net XA40: J540.1 (Pin_1)
- new net XA41: J541.1 (Pin_1)
- new net XA42: J542.1 (Pin_1)
- new net XA43: J543.1 (Pin_1)
- new net XA44: J544.1 (Pin_1)
- new net XA45: J545.1 (Pin_1)
- new net XA46: J546.1 (Pin_1)
- new net XA47: J547.1 (Pin_1)
- new net XA48: J548.1 (Pin_1)
- new net XA49: J549.1 (Pin_1)
- new net XA5: J505.1 (Pin_1)
- new net XA50: J550.1 (Pin_1)
- new net XA51: J551.1 (Pin_1)
- new net XA52: J552.1 (Pin_1)
- new net XA53: J553.1 (Pin_1)
- new net XA54: J554.1 (Pin_1)
- new net XA55: J555.1 (Pin_1)
- new net XA56: J556.1 (Pin_1)
- new net XA57: J557.1 (Pin_1)
- new net XA58: J558.1 (Pin_1)
- new net XA59: J559.1 (Pin_1)
- new net XA6: J506.1 (Pin_1)
- new net XA60: J560.1 (Pin_1)
- new net XA61: J561.1 (Pin_1)
- new net XA62: J562.1 (Pin_1)
- new net XA63: J563.1 (Pin_1)
- new net XA7: J507.1 (Pin_1)
- new net XA8: J508.1 (Pin_1)
- new net XA9: J509.1 (Pin_1)
- new net XB10: J574.1 (Pin_1)
- new net XB11: J575.1 (Pin_1)
- new net XB12: J576.1 (Pin_1)
- new net XB13: J577.1 (Pin_1)
- new net XB14: J578.1 (Pin_1)
- new net XB15: J579.1 (Pin_1)
- new net XB16: J580.1 (Pin_1)
- new net XB17: J581.1 (Pin_1)
- new net XB18: J582.1 (Pin_1)
- new net XB19: J583.1 (Pin_1)
- new net XB2: J566.1 (Pin_1)
- new net XB20: J584.1 (Pin_1)
- new net XB21: J585.1 (Pin_1)
- new net XB22: J586.1 (Pin_1)
- new net XB23: J587.1 (Pin_1)
- new net XB24: J588.1 (Pin_1)
- new net XB25: J589.1 (Pin_1)
- new net XB26: J590.1 (Pin_1)
- new net XB27: J591.1 (Pin_1)
- new net XB28: J592.1 (Pin_1)
- new net XB29: J593.1 (Pin_1)
- new net XB3: J567.1 (Pin_1)
- new net XB30: J594.1 (Pin_1)
- new net XB31: J595.1 (Pin_1)
- new net XB32: J596.1 (Pin_1)
- new net XB33: J597.1 (Pin_1)
- new net XB34: J598.1 (Pin_1)
- new net XB35: J599.1 (Pin_1)
- new net XB36: J600.1 (Pin_1)
- new net XB37: J601.1 (Pin_1)
- new net XB38: J602.1 (Pin_1)
- new net XB39: J603.1 (Pin_1)
- new net XB4: J568.1 (Pin_1)
- new net XB40: J604.1 (Pin_1)
- new net XB41: J605.1 (Pin_1)
- new net XB42: J606.1 (Pin_1)
- new net XB43: J607.1 (Pin_1)
- new net XB44: J608.1 (Pin_1)
- new net XB45: J609.1 (Pin_1)
- new net XB46: J610.1 (Pin_1)
- new net XB47: J611.1 (Pin_1)
- new net XB48: J612.1 (Pin_1)
- new net XB49: J613.1 (Pin_1)
- new net XB5: J569.1 (Pin_1)
- new net XB50: J614.1 (Pin_1)
- new net XB51: J615.1 (Pin_1)
- new net XB52: J616.1 (Pin_1)
- new net XB53: J617.1 (Pin_1)
- new net XB54: J618.1 (Pin_1)
- new net XB55: J619.1 (Pin_1)
- new net XB56: J620.1 (Pin_1)
- new net XB57: J621.1 (Pin_1)
- new net XB58: J622.1 (Pin_1)
- new net XB59: J623.1 (Pin_1)
- new net XB6: J570.1 (Pin_1)
- new net XB60: J624.1 (Pin_1)
- new net XB61: J625.1 (Pin_1)
- new net XB62: J626.1 (Pin_1)
- new net XB63: J627.1 (Pin_1)
- new net XB7: J571.1 (Pin_1)
- new net XB8: J572.1 (Pin_1)
- new net XB9: J573.1 (Pin_1)
- new net YA10: J638.1 (Pin_1)
- new net YA11: J639.1 (Pin_1)
- new net YA12: J640.1 (Pin_1)
- new net YA13: J641.1 (Pin_1)
- new net YA14: J642.1 (Pin_1)
- new net YA15: J643.1 (Pin_1)
- new net YA16: J644.1 (Pin_1)
- new net YA17: J645.1 (Pin_1)
- new net YA18: J646.1 (Pin_1)
- new net YA19: J647.1 (Pin_1)
- new net YA2: J630.1 (Pin_1)
- new net YA20: J648.1 (Pin_1)
- new net YA21: J649.1 (Pin_1)
- new net YA22: J650.1 (Pin_1)
- new net YA23: J651.1 (Pin_1)
- new net YA24: J652.1 (Pin_1)
- new net YA25: J653.1 (Pin_1)
- new net YA26: J654.1 (Pin_1)
- new net YA27: J655.1 (Pin_1)
- new net YA28: J656.1 (Pin_1)
- new net YA29: J657.1 (Pin_1)
- new net YA3: J631.1 (Pin_1)
- new net YA30: J658.1 (Pin_1)
- new net YA31: J659.1 (Pin_1)
- new net YA32: J660.1 (Pin_1)
- new net YA33: J661.1 (Pin_1)
- new net YA34: J662.1 (Pin_1)
- new net YA35: J663.1 (Pin_1)
- new net YA36: J664.1 (Pin_1)
- new net YA37: J665.1 (Pin_1)
- new net YA38: J666.1 (Pin_1)
- new net YA39: J667.1 (Pin_1)
- new net YA4: J632.1 (Pin_1)
- new net YA40: J668.1 (Pin_1)
- new net YA41: J669.1 (Pin_1)
- new net YA42: J670.1 (Pin_1)
- new net YA43: J671.1 (Pin_1)
- new net YA44: J672.1 (Pin_1)
- new net YA45: J673.1 (Pin_1)
- new net YA46: J674.1 (Pin_1)
- new net YA47: J675.1 (Pin_1)
- new net YA48: J676.1 (Pin_1)
- new net YA49: J677.1 (Pin_1)
- new net YA5: J633.1 (Pin_1)
- new net YA50: J678.1 (Pin_1)
- new net YA51: J679.1 (Pin_1)
- new net YA52: J680.1 (Pin_1)
- new net YA53: J681.1 (Pin_1)
- new net YA54: J682.1 (Pin_1)
- new net YA55: J683.1 (Pin_1)
- new net YA56: J684.1 (Pin_1)
- new net YA57: J685.1 (Pin_1)
- new net YA58: J686.1 (Pin_1)
- new net YA59: J687.1 (Pin_1)
- new net YA6: J634.1 (Pin_1)
- new net YA60: J688.1 (Pin_1)
- new net YA61: J689.1 (Pin_1)
- new net YA62: J690.1 (Pin_1)
- new net YA63: J691.1 (Pin_1)
- new net YA7: J635.1 (Pin_1)
- new net YA8: J636.1 (Pin_1)
- new net YA9: J637.1 (Pin_1)
- new net YB10: J702.1 (Pin_1)
- new net YB11: J703.1 (Pin_1)
- new net YB12: J704.1 (Pin_1)
- new net YB13: J705.1 (Pin_1)
- new net YB14: J706.1 (Pin_1)
- new net YB15: J707.1 (Pin_1)
- new net YB16: J708.1 (Pin_1)
- new net YB17: J709.1 (Pin_1)
- new net YB18: J710.1 (Pin_1)
- new net YB19: J711.1 (Pin_1)
- new net YB2: J694.1 (Pin_1)
- new net YB20: J712.1 (Pin_1)
- new net YB21: J713.1 (Pin_1)
- new net YB22: J714.1 (Pin_1)
- new net YB23: J715.1 (Pin_1)
- new net YB24: J716.1 (Pin_1)
- new net YB25: J717.1 (Pin_1)
- new net YB26: J718.1 (Pin_1)
- new net YB27: J719.1 (Pin_1)
- new net YB28: J720.1 (Pin_1)
- new net YB29: J721.1 (Pin_1)
- new net YB3: J695.1 (Pin_1)
- new net YB30: J722.1 (Pin_1)
- new net YB31: J723.1 (Pin_1)
- new net YB32: J724.1 (Pin_1)
- new net YB33: J725.1 (Pin_1)
- new net YB34: J726.1 (Pin_1)
- new net YB35: J727.1 (Pin_1)
- new net YB36: J728.1 (Pin_1)
- new net YB37: J729.1 (Pin_1)
- new net YB38: J730.1 (Pin_1)
- new net YB39: J731.1 (Pin_1)
- new net YB4: J696.1 (Pin_1)
- new net YB40: J732.1 (Pin_1)
- new net YB41: J733.1 (Pin_1)
- new net YB42: J734.1 (Pin_1)
- new net YB43: J735.1 (Pin_1)
- new net YB44: J736.1 (Pin_1)
- new net YB45: J737.1 (Pin_1)
- new net YB46: J738.1 (Pin_1)
- new net YB47: J739.1 (Pin_1)
- new net YB48: J740.1 (Pin_1)
- new net YB49: J741.1 (Pin_1)
- new net YB5: J697.1 (Pin_1)
- new net YB50: J742.1 (Pin_1)
- new net YB51: J743.1 (Pin_1)
- new net YB52: J744.1 (Pin_1)
- new net YB53: J745.1 (Pin_1)
- new net YB54: J746.1 (Pin_1)
- new net YB55: J747.1 (Pin_1)
- new net YB56: J748.1 (Pin_1)
- new net YB57: J749.1 (Pin_1)
- new net YB58: J750.1 (Pin_1)
- new net YB59: J751.1 (Pin_1)
- new net YB6: J698.1 (Pin_1)
- new net YB60: J752.1 (Pin_1)
- new net YB61: J753.1 (Pin_1)
- new net YB62: J754.1 (Pin_1)
- new net YB63: J755.1 (Pin_1)
- new net YB7: J699.1 (Pin_1)
- new net YB8: J700.1 (Pin_1)
- new net YB9: J701.1 (Pin_1)
- no-connect marks 8 -> 1
Other:
- sheet CCS renamed CCS X
- sheet Decode Block renamed X FWD
- sheet Drive Block renamed X0 FWD
- added sheet CCS INH (ccs.kicad_sch)
- added sheet CCS Y (ccs.kicad_sch)
- added sheet Decode CTRL Y (decode_ctrl_y.kicad_sch)
- added sheet Steer 2x2 (steer_2x2.kicad_sch)
- added sheet X REV (decode_block.kicad_sch)
- added sheet X0 REV (drive_block.kicad_sch)
- added sheet X1 FWD (drive_block.kicad_sch)
- added sheet X1 REV (drive_block.kicad_sch)
- added sheet X2 FWD (drive_block.kicad_sch)
- added sheet X2 REV (drive_block.kicad_sch)
- added sheet X3 FWD (drive_block.kicad_sch)
- added sheet X3 REV (drive_block.kicad_sch)
- added sheet X4 FWD (drive_block.kicad_sch)
- added sheet X4 REV (drive_block.kicad_sch)
- added sheet X5 FWD (drive_block.kicad_sch)
- added sheet X5 REV (drive_block.kicad_sch)
- added sheet X6 FWD (drive_block.kicad_sch)
- added sheet X6 REV (drive_block.kicad_sch)
- added sheet X7 FWD (drive_block.kicad_sch)
- added sheet X7 REV (drive_block.kicad_sch)
- added sheet Y FWD (decode_block.kicad_sch)
- added sheet Y REV (decode_block.kicad_sch)
- added sheet Y0 FWD (drive_block.kicad_sch)
- added sheet Y0 REV (drive_block.kicad_sch)
- added sheet Y1 FWD (drive_block.kicad_sch)
- added sheet Y1 REV (drive_block.kicad_sch)
- added sheet Y2 FWD (drive_block.kicad_sch)
- added sheet Y2 REV (drive_block.kicad_sch)
- added sheet Y3 FWD (drive_block.kicad_sch)
- added sheet Y3 REV (drive_block.kicad_sch)
- added sheet Y4 FWD (drive_block.kicad_sch)
- added sheet Y4 REV (drive_block.kicad_sch)
- added sheet Y5 FWD (drive_block.kicad_sch)
- added sheet Y5 REV (drive_block.kicad_sch)
- added sheet Y6 FWD (drive_block.kicad_sch)
- added sheet Y6 REV (drive_block.kicad_sch)
- added sheet Y7 FWD (drive_block.kicad_sch)
- added sheet Y7 REV (drive_block.kicad_sch)
- sheet Decode CTRL ports: added ADDR_NH0, ADDR_NH1, ADDR_NH2, ADDR_NL0, ADDR_NL1, ADDR_NL2, BANK_EN; removed ADDR_XH0, ADDR_XH1, ADDR_XH2, ADDR_XL0, ADDR_XL1, ADDR_XL2, ADDR_YH0, ADDR_YH1, ADDR_YH2, ADDR_YL0, ADDR_YL1, ADDR_YL2, FWD_EN_n
- sheet X0 FWD ports: added N_HS_OUT, N_LS_OUT; removed NAn, NBn
- note added: "DECODE — four decode_block calls (X/Y, FWD/REV); ADDR_Y and REV_EN_n are driven"
- note added: "DRIVE — eight drive_block calls (groups 0 and 1, X and Y, FWD and REV) plus steer_2x2"
- note added: "RP2040 timing header. These nets are the e2e stimulus."
- note removed: "DECODE — Decode Block (N=axis, n=HS/LS bank); X FWD wired for 1×1 bring-up"
- note removed: "DRIVE — Drive Block (N=axis, n=line); X0 FWD wired for 1×1 bring-up"
