File: kicad/core/core.kicad_sch (KiCad schematic)
At the start: 273 parts, among them J400 PIO, J401 PIO, J402 PIO, J403 PIO, J404 PIO, J405 PIO, J406 PIO, J407 PIO, J408 PIO, J409 PIO, J410 PIO, J411 PIO, J412 PIO, J413 PIO, J414 PIO, J415 PIO, J416 PIO, J500 Edge, J501 Edge, J502 Edge, J503 Edge, J504 Edge, J505 Edge, J506 Edge, J507 Edge, J508 Edge, J509 Edge, J510 Edge, J511 Edge, J512 Edge, J513 Edge, J514 Edge, J515 Edge, J516 Edge, J517 Edge, J518 Edge, J519 Edge, J520 Edge, J521 Edge, J522 Edge, J523 Edge, J524 Edge, J525 Edge, J526 Edge, J527 Edge, J528 Edge, J529 Edge, J530 Edge, J531 Edge, J532 Edge, J533 Edge, J534 Edge, J535 Edge, J536 Edge, J537 Edge, J538 Edge, J539 Edge, J540 Edge, J541 Edge, J542 Edge, J543 Edge, J544 Edge, J545 Edge, J546 Edge, J547 Edge, J548 Edge, J549 Edge, J550 Edge, J551 Edge, J552 Edge, J553 Edge, J554 Edge, J555 Edge, J556 Edge, J557 Edge, J558 Edge, J559 Edge, J560 Edge, J561 Edge, J562 Edge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

Commit message: Scaled to 64x64 and paying heavy due. We can learn if we have to... I guess.
Other:
- sheet Steer 2x2 renamed Steer 64
- sheet Magnetic Cores: file magnetic_core_2x2.kicad_sch -> magnetic_core_64x64.kicad_sch
- sheet Magnetic Cores ports: added XA10, XA11, XA12, XA13, XA14, XA15, XA16, XA17, XA18, XA19, XA2, XA20, XA21, XA22, XA23, XA24, XA25, XA26, XA27, XA28, XA29, XA3, XA30, XA31, XA32, XA33, XA34, XA35, XA36, XA37, XA38, XA39, XA4, XA40, XA41, XA42, XA43, XA44, XA45, XA46, XA47, XA48, XA49, XA5, XA50, XA51, XA52, XA53, XA54, XA55, XA56, XA57, XA58, XA59, XA6, XA60, XA61, XA62, XA63, XA7, XA8, XA9, XB10, XB11, XB12, XB13, XB14, XB15, XB16, XB17, XB18, XB19, XB2, XB20, XB21, XB22, XB23, XB24, XB25, XB26, XB27, XB28, XB29, XB3, XB30, XB31, XB32, XB33, XB34, XB35, XB36, XB37, XB38, XB39, XB4, XB40, XB41, XB42, XB43, XB44, XB45, XB46, XB47, XB48, XB49, XB5, XB50, XB51, XB52, XB53, XB54, XB55, XB56, XB57, XB58, XB59, XB6, XB60, XB61, XB62, XB63, XB7, XB8, XB9, YA10, YA11, YA12, YA13, YA14, YA15, YA16, YA17, YA18, YA19, YA2, YA20, YA21, YA22, YA23, YA24, YA25, YA26, YA27, YA28, YA29, YA3, YA30, YA31, YA32, YA33, YA34, YA35, YA36, YA37, YA38, YA39, YA4, YA40, YA41, YA42, YA43, YA44, YA45, YA46, YA47, YA48, YA49, YA5, YA50, YA51, YA52, YA53, YA54, YA55, YA56, YA57, YA58, YA59, YA6, YA60, YA61, YA62, YA63, YA7, YA8, YA9, YB10, YB11, YB12, YB13, YB14, YB15, YB16, YB17, YB18, YB19, YB2, YB20, YB21, YB22, YB23, YB24, YB25, YB26, YB27, YB28, YB29, YB3, YB30, YB31, YB32, YB33, YB34, YB35, YB36, YB37, YB38, YB39, YB4, YB40, YB41, YB42, YB43, YB44, YB45, YB46, YB47, YB48, YB49, YB5, YB50, YB51, YB52, YB53, YB54, YB55, YB56, YB57, YB58, YB59, YB6, YB60, YB61, YB62, YB63, YB7, YB8, YB9; removed none
- sheet Steer 64: file steer_2x2.kicad_sch -> steer_64.kicad_sch
- note added: "DRIVE — 32 drive_block calls (groups 0-7, X and Y, FWD and REV) plus steer_64"
- note removed: "DRIVE — eight drive_block calls (groups 0 and 1, X and Y, FWD and REV) plus steer_2x2"
