File: kicad/core/decoupling_logic.kicad_sch (KiCad schematic)
At the start: 6 parts

Commit message: Prove the 2×2 access cycle from the address pins through decode, drive, and the sense latch.
Three current sinks, the diode matrix, and drive groups 0--7 are on the schematic. The four-core decks are the gate; weave inductance is still an open input.
Parts:
- removed C5: 100n, Capacitor_SMD:C_0805_2012Metric, symbol Device:C
- removed C6: 1u, Capacitor_SMD:C_0805_2012Metric, symbol Device:C
Other:
- note added: "Decode Block carries its own +3V3 100n per IC. CCS carries its own +5V pair."
- note added: "Logic decoupling — +3V3 (Sense / Latch)"
- note removed: "CCS U3 (OPA192) +5V"
- note removed: "Decode Block carries its own +3V3 100n per IC"
- note removed: "Logic decoupling — +3V3 / +5V (shared Sense / Latch / CCS)"
